File: modules/alu/alu.kicad_pcb (KiCad board)
At the start: 2 copper layers, 1978 parts, among them Q1 2N3906, Q10 2N3904, Q100 2N3904, Q101 2N3904, Q102 2N3904, Q103 2N3906, Q104 2N3904, Q105 2N3906, Q106 2N3904, Q107 2N3906, Q108 2N3904, Q109 2N3906, Q11 2N3904, Q110 2N3906, Q111 2N3906, Q112 2N3904, Q113 2N3906, Q114 2N3906, Q115 2N3906, Q116 2N3906, Q117 2N3904, Q118 2N3906, Q119 2N3906, Q12 2N3904, Q120 2N3906, Q121 2N3906, Q122 2N3904, Q123 2N3904, Q124 2N3904, Q125 2N3904, Q126 2N3904, Q127 2N3904, Q128 2N3904, Q129 2N3904, Q13 2N3904, Q130 2N3904, Q131 2N3904, Q132 2N3904, Q133 2N3904, Q134 2N3904, Q135 2N3904, Q136 2N3904, Q137 2N3906, Q138 2N3906, Q139 2N3906, Q14 2N3904, Q140 2N3906, Q141 2N3904, Q142 2N3904, Q143 2N3904, Q144 2N3906, Q145 2N3904, Q146 2N3904, Q147 2N3906, Q148 2N3904, Q149 2N3904, Q15 2N3904, Q150 2N3904, Q151 2N3904, Q152 2N3904, Q153 2N3906, Q154 2N3904, Q155 2N3906, Q156 2N3904, Q157 2N3906, Q158 2N3904, Q159 2N3906, Q16 2N3904, Q160 2N3906, Q161 2N3906, Q162 2N3904, Q163 2N3906, Q164 2N3906, Q165 2N3906, Q166 2N3906, Q167 2N3904, Q168 2N3906, Q169 2N3906, Q17 2N3904, Q170 2N3906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

Commit message: Some fixes to the ALU schematics
Parts:
- removed D1, D10, D100, D101, D102, D103, D104, D105, D106, D107, D108, D109, D11, D110, D111, D112, D113, D114, D115, D116, D117, D118, D119, D12, D120, D121, D122, D123, D124, D125, D126, D127, D128, D129, D13, D130, D131, D132, D133, D134, D135, D136, D137, D138, D139, D14, D140, D141, D142, D143, D144, D145, D146, D147, D148, D149, D15, D150, D151, D152, D153, D154, D155, D156, D157, D158, D159, D16, D160, D161, D162, D163, D164, D165, D166, D167, D168, D169, D17, D170, D171, D172, D173, D174, D175, D176, D177, D178, D179, D18, D180, D181, D182, D183, D184, D185, D186, D187, D188, D189, D19, D190, D191, D192, D193, D194, D195, D196, D197, D198, D199, D2, D20, D200, D201, D202, D203, D204, D205, D206, D207, D208, D209, D21, D210, D211, D212, D213, D214, D215, D216, D217, D218, D219, D22, D220, D221, D222, D223, D224, D225, D226, D227, D228, D229, D23, D230, D231, D232, D233, D234, D24, D25, D26, D27, D28, D29, D3, D30, D31, D32, D33, D34, D35, D36, D37, D38, D39, D4, D40, D41, D42, D43, D44, D45, D46, D47, D48, D49, D5, D50, D51, D52, D53, D54, D55, D56, D57, D58, D59, D6, D60, D61, D62, D63, D64, D65, D66, D67, D68, D69, D7, D70, D71, D72, D73, D74, D75, D76, D77, D78, D79, D8, D80, D81, D82, D83, D84, D85, D86, D87, D88, D89, D9, D90, D91, D92, D93, D94, D95, D96, D97, D98, D99: BAT54W, Package_TO_SOT_SMD:SOT-323_SC-70
- removed Q1, Q103, Q105, Q107, Q109, Q110, Q111, Q113, Q114, Q115, Q116, Q118, Q119, Q120, Q121, Q137, Q138, Q139, Q140, Q144, Q147, Q153, Q155, Q157, Q159, Q160, Q161, Q163, Q164, Q165, Q166, Q168, Q169, Q170, Q171, Q187, Q188, Q189, Q190, Q194, Q197, Q2, Q203, Q205, Q207, Q209, Q210, Q211, Q213, Q214, Q215, Q216, Q218, Q219, Q220, Q221, Q229, Q230, Q231, Q232, Q233, Q234, Q235, Q236, Q25, Q253, Q254, Q255, Q256, Q26, Q265, Q266, Q267, Q268, Q27, Q272, Q275, Q28, Q281, Q283, Q285, Q287, Q288, Q289, Q291, Q292, Q293, Q294, Q296, Q297, Q298, Q299, Q3, Q315, Q316, Q317, Q318, Q322, Q325, Q331, Q333, Q335, Q337, Q338, Q339, Q341, Q342, Q343, Q344, Q346, Q347, Q348, Q349, Q365, Q366, Q367, Q368, Q37, Q372, Q375, Q38, Q381, Q383, Q385, Q387, Q388, Q389, Q39, Q391, Q392, Q393, Q394, Q396, Q397, Q398, Q399, Q4, Q40, Q415, Q416, Q417, Q418, Q422, Q425, Q431, Q433, Q435, Q437, Q438, Q439, Q44, Q441, Q442, Q443, Q444, Q446, Q447, Q448, Q449, Q457, Q458, Q459, Q460, Q461, Q462, Q463, Q464, Q47, Q481, Q482, Q483, Q484, Q493, Q494, Q495, Q496, Q5, Q500, Q503, Q509, Q511, Q513, Q515, Q516, Q517, Q519, Q520, Q521, Q522, Q524, Q525, Q526, Q527, Q53, Q543, Q544, Q545, Q546, Q55, Q550, Q553, Q559, Q561, Q563, Q565, Q566, Q567, Q569, Q57, Q570, Q571, Q572, Q574, Q575, Q576, Q577, Q59, Q593, Q594, Q595, Q596, Q6, Q60, Q600, Q603, Q609, Q61, Q611, Q613, Q615, Q616, Q617, Q619, Q620, Q621, Q622, Q624, Q625, Q626, Q627, Q63, Q64, Q643, Q644, Q645, Q646, Q65, Q650, Q653, Q659, Q66, Q661, Q663, Q665, Q666, Q667, Q669, Q670, Q671, Q672, Q674, Q675, Q676, Q677, Q68, Q685, Q686, Q687, Q688, Q689, Q69, Q690, Q691, Q692, Q7, Q70, Q709, Q71, Q710, Q711, Q712, Q721, Q722, Q723, Q724, Q728, Q731, Q737, Q739, Q741, Q743, Q744, Q745, Q747, Q748, Q749, Q750, Q752, Q753, Q754, Q755, Q771, Q772, Q773, Q774, Q778, Q781, Q787, Q789, Q791, Q793, Q794, Q795, Q797, Q798, Q799, Q8, Q800, Q802, Q803, Q804, Q805, Q821, Q822, Q823, Q824, Q828, Q831, Q837, Q839, Q841, Q843, Q844, Q845, Q847, Q848, Q849, Q850, Q852, Q853, Q854, Q855, Q87, Q871, Q872, Q873, Q874, Q878, Q88, Q881, Q887, Q889, Q89, Q891, Q893, Q894, Q895, Q897, Q898, Q899, Q90, Q900, Q902, Q903, Q904, Q905, Q916, Q917, Q94, Q944, Q945, Q952, Q953, Q958, Q959, Q960, Q97: 2N3906, Package_TO_SOT_SMD:SOT-23-3
- removed Q10, Q100, Q101, Q102, Q104, Q106, Q108, Q11, Q112, Q117, Q12, Q122, Q123, Q124, Q125, Q126, Q127, Q128, Q129, Q13, Q130, Q131, Q132, Q133, Q134, Q135, Q136, Q14, Q141, Q142, Q143, Q145, Q146, Q148, Q149, Q15, Q150, Q151, Q152, Q154, Q156, Q158, Q16, Q162, Q167, Q17, Q172, Q173, Q174, Q175, Q176, Q177, Q178, Q179, Q18, Q180, Q181, Q182, Q183, Q184, Q185, Q186, Q19, Q191, Q192, Q193, Q195, Q196, Q198, Q199, Q20, Q200, Q201, Q202, Q204, Q206, Q208, Q21, Q212, Q217, Q22, Q222, Q223, Q224, Q225, Q226, Q227, Q228, Q23, Q237, Q238, Q239, Q24, Q240, Q241, Q242, Q243, Q244, Q245, Q246, Q247, Q248, Q249, Q250, Q251, Q252, Q257, Q258, Q259, Q260, Q261, Q262, Q263, Q264, Q269, Q270, Q271, Q273, Q274, Q276, Q277, Q278, Q279, Q280, Q282, Q284, Q286, Q29, Q290, Q295, Q30, Q300, Q301, Q302, Q303, Q304, Q305, Q306, Q307, Q308, Q309, Q31, Q310, Q311, Q312, Q313, Q314, Q319, Q32, Q320, Q321, Q323, Q324, Q326, Q327, Q328, Q329, Q33, Q330, Q332, Q334, Q336, Q34, Q340, Q345, Q35, Q350, Q351, Q352, Q353, Q354, Q355, Q356, Q357, Q358, Q359, Q36, Q360, Q361, Q362, Q363, Q364, Q369, Q370, Q371, Q373, Q374, Q376, Q377, Q378, Q379, Q380, Q382, Q384, Q386, Q390, Q395, Q400, Q401, Q402, Q403, Q404, Q405, Q406, Q407, Q408, Q409, Q41, Q410, Q411, Q412, Q413, Q414, Q419, Q42, Q420, Q421, Q423, Q424, Q426, Q427, Q428, Q429, Q43, Q430, Q432, Q434, Q436, Q440, Q445, Q45, Q450, Q451, Q452, Q453, Q454, Q455, Q456, Q46, Q465, Q466, Q467, Q468, Q469, Q470, Q471, Q472, Q473, Q474, Q475, Q476, Q477, Q478, Q479, Q48, Q480, Q485, Q486, Q487, Q488, Q489, Q49, Q490, Q491, Q492, Q497, Q498, Q499, Q50, Q501, Q502, Q504, Q505, Q506, Q507, Q508, Q51, Q510, Q512, Q514, Q518, Q52, Q523, Q528, Q529, Q530, Q531, Q532, Q533, Q534, Q535, Q536, Q537, Q538, Q539, Q54, Q540, Q541, Q542, Q547, Q548, Q549, Q551, Q552, Q554, Q555, Q556, Q557, Q558, Q56, Q560, Q562, Q564, Q568, Q573, Q578, Q579, Q58, Q580, Q581, Q582, Q583, Q584, Q585, Q586, Q587, Q588, Q589, Q590, Q591, Q592, Q597, Q598, Q599, Q601, Q602, Q604, Q605, Q606, Q607, Q608, Q610, Q612, Q614, Q618, Q62, Q623, Q628, Q629, Q630, Q631, Q632, Q633, Q634, Q635, Q636, Q637, Q638, Q639, Q640, Q641, Q642, Q647, Q648, Q649, Q651, Q652, Q654, Q655, Q656, Q657, Q658, Q660, Q662, Q664, Q668, Q67, Q673, Q678, Q679, Q680, Q681, Q682, Q683, Q684, Q693, Q694, Q695, Q696, Q697, Q698, Q699, Q700, Q701, Q702, Q703, Q704, Q705, Q706, Q707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: 2N3904, Package_TO_SOT_SMD:SOT-23-3
- removed R1, R100, R115, R116, R118, R134, R136, R139, R141, R156, R157, R159, R175, R177, R180, R182, R189, R190, R191, R192, R2, R221, R222, R224, R240, R242, R245, R247, R262, R263, R265, R281, R283, R286, R288, R3, R303, R304, R306, R322, R324, R327, R329, R33, R34, R344, R345, R347, R36, R363, R365, R368, R370, R385, R386, R387, R388, R4, R417, R418, R420, R436, R438, R441, R443, R458, R459, R461, R477, R479, R482, R484, R499, R500, R502, R518, R52, R520, R523, R525, R54, R540, R541, R543, R559, R561, R564, R566, R57, R573, R574, R575, R576, R59, R605, R606, R608, R624, R626, R629, R631, R646, R647, R649, R665, R667, R670, R672, R687, R688, R690, R706, R708, R711, R713, R728, R729, R731, R74, R747, R749, R75, R752, R754, R77, R788, R810, R817, R93, R95, R98: 520, Resistor_SMD:R_0603_1608Metric_Pad0.98x0.95mm_HandSolder
- removed R10, R101, R102, R103, R104, R107, R108, R109, R11, R110, R113, R114, R119, R12, R120, R121, R122, R125, R126, R130, R131, R132, R133, R142, R143, R144, R145, R148, R149, R150, R151, R154, R155, R160, R161, R162, R163, R166, R167, R171, R172, R173, R174, R183, R184, R185, R186, R193, R194, R195, R196, R197, R198, R199, R200, R213, R214, R215, R216, R219, R220, R225, R226, R227, R228, R231, R232, R236, R237, R238, R239, R248, R249, R25, R250, R251, R254, R255, R256, R257, R26, R260, R261, R266, R267, R268, R269, R27, R272, R273, R277, R278, R279, R28, R280, R289, R290, R291, R292, R295, R296, R297, R298, R301, R302, R307, R308, R309, R31, R310, R313, R314, R318, R319, R32, R320, R321, R330, R331, R332, R333, R336, R337, R338, R339, R342, R343, R348, R349, R350, R351, R354, R355, R359, R360, R361, R362, R37, R371, R372, R373, R374, R38, R389, R39, R390, R391, R392, R393, R394, R395, R396, R40, R409, R410, R411, R412, R415, R416, R421, R422, R423, R424, R427, R428, R43, R432, R433, R434, R435, R44, R444, R445, R446, R447, R450, R451, R452, R453, R456, R457, R462, R463, R464, R465, R468, R469, R473, R474, R475, R476, R48, R485, R486, R487, R488, R49, R491, R492, R493, R494, R497, R498, R5, R50, R503, R504, R505, R506, R509, R51, R510, R514, R515, R516, R517, R526, R527, R528, R529, R532, R533, R534, R535, R538, R539, R544, R545, R546, R547, R550, R551, R555, R556, R557, R558, R567, R568, R569, R570, R577, R578, R579, R580, R581, R582, R583, R584, R597, R598, R599, R6, R60, R600, R603, R604, R609, R61, R610, R611, R612, R615, R616, R62, R620, R621, R622, R623, R63, R632, R633, R634, R635, R638, R639, R640, R641, R644, R645, R650, R651, R652, R653, R656, R657, R66, R661, R662, R663, R664, R67, R673, R674, R675, R676, R679, R68, R680, R681, R682, R685, R686, R69, R691, R692, R693, R694, R697, R698, R7, R702, R703, R704, R705, R714, R715, R716, R717, R72, R720, R721, R722, R723, R726, R727, R73, R732, R733, R734, R735, R738, R739, R743, R744, R745, R746, R755, R756, R757, R758, R78, R785, R786, R789, R79, R790, R8, R80, R801, R802, R804, R805, R807, R808, R81, R811, R812, R814, R815, R818, R819, R821, R822, R84, R85, R89, R9, R90, R91, R92: 220, Resistor_SMD:R_0603_1608Metric_Pad0.98x0.95mm_HandSolder
- removed R105, R106, R111, R112, R117, R123, R124, R127, R128, R129, R13, R135, R137, R138, R14, R140, R146, R147, R15, R152, R153, R158, R16, R164, R165, R168, R169, R17, R170, R176, R178, R179, R18, R181, R187, R188, R19, R20, R201, R202, R203, R204, R205, R206, R207, R208, R209, R21, R210, R211, R212, R217, R218, R22, R223, R229, R23, R230, R233, R234, R235, R24, R241, R243, R244, R246, R252, R253, R258, R259, R264, R270, R271, R274, R275, R276, R282, R284, R285, R287, R29, R293, R294, R299, R30, R300, R305, R311, R312, R315, R316, R317, R323, R325, R326, R328, R334, R335, R340, R341, R346, R35, R352, R353, R356, R357, R358, R364, R366, R367, R369, R375, R376, R397, R398, R399, R400, R401, R402, R403, R404, R405, R406, R407, R408, R41, R413, R414, R419, R42, R425, R426, R429, R430, R431, R437, R439, R440, R442, R448, R449, R45, R454, R455, R46, R460, R466, R467, R47, R470, R471, R472, R478, R480, R481, R483, R489, R490, R495, R496, R501, R507, R508, R511, R512, R513, R519, R521, R522, R524, R53, R530, R531, R536, R537, R542, R548, R549, R55, R552, R553, R554, R56, R560, R562, R563, R565, R571, R572, R58, R585, R586, R587, R588, R589, R590, R591, R592, R593, R594, R595, R596, R601, R602, R607, R613, R614, R617, R618, R619, R625, R627, R628, R630, R636, R637, R64, R642, R643, R648, R65, R654, R655, R658, R659, R660, R666, R668, R669, R671, R677, R678, R683, R684, R689, R695, R696, R699, R70, R700, R701, R707, R709, R71, R710, R712, R718, R719, R724, R725, R730, R736, R737, R740, R741, R742, R748, R750, R751, R753, R759, R76, R760, R787, R791, R803, R806, R809, R813, R816, R82, R820, R823, R824, R825, R83, R86, R87, R88, R94, R96, R97, R99: 100, Resistor_SMD:R_0603_1608Metric_Pad0.98x0.95mm_HandSolder
