File: modules/alu/alu.kicad_sch (KiCad schematic)
At the start: 20 parts, among them Q12 2N3904, Q13 2N3904, Q14 2N3904, Q2 2N3904, Q3 2N3904, Q4 2N3904, Q6 2N3906, Q7 2N3906

Commit message: Much work towards an actual ALU bit-cell.
Parts:
- removed Q6: 2N3906, Package_TO_SOT_SMD:SOT-23-3, symbol Simulation_SPICE:PNP
- added D10, D11, D3, D4, D5, D6, D7, D8, D9: BAT54W, Package_TO_SOT_SMD:SOT-323_SC-70, symbol Diode:BAT54W
- added Q1, Q11, Q15, Q16, Q17, Q19, Q21, Q23, Q28, Q29, Q30, Q33, Q34, Q36, Q43, Q44, Q45, Q5, Q6: 2N3904, Package_TO_SOT_SMD:SOT-23-3, symbol Simulation_SPICE:NPN
- added Q10, Q18, Q20, Q22, Q24, Q25, Q26, Q27, Q31, Q32, Q35, Q37, Q38, Q39, Q40, Q41, Q42, Q8, Q9: 2N3906, Package_TO_SOT_SMD:SOT-23-3, symbol Simulation_SPICE:PNP
- added R11, R12, R13, R14, R17, R18, R19, R20, R24, R25, R27, R28, R29, R30, R34, R35, R37, R38, R4, R6: 220, Resistor_SMD:R_0603_1608Metric_Pad0.98x0.95mm_HandSolder, symbol Device:R_Small_US
- added R15, R16, R21, R22, R26, R31, R32, R36, R39, R7: 100, Resistor_SMD:R_0603_1608Metric_Pad0.98x0.95mm_HandSolder, symbol Device:R_Small_US
- added R23, R33: 520, Resistor_SMD:R_0603_1608Metric_Pad0.98x0.95mm_HandSolder, symbol Device:R_Small_US
- added V4: VPULSE, symbol Simulation_SPICE:VPULSE
- R1, R2: value 220 -> 10k
- R10: value 100 -> 520
- R3: value 100 -> 220
- R5: value 520 -> 220
- R8: value 220 -> 100
- R9: value 220 -> 520
Connections:
- net 0: now also R1.2, Q10.1 (C), Q15.3 (E), Q16.3 (E), Q18.1 (C), Q20.1 (C), Q22.1 (C), Q23.3 (E), Q25.1 (C), Q26.1 (C), Q27.1 (C), Q30.3 (E), Q31.1 (C), Q32.1 (C), Q36.3 (E), Q37.1 (C), Q38.1 (C), Q39.1 (C), Q40.1 (C), Q41.1 (C), Q45.3 (E), Q5.3 (E), Q6.3 (E), Q8.1 (C), Q9.1 (C), R12.2, R14.2, R18.2, R22.2, R25.2, R30.2, R31.2, R36.2, R38.2, R4.2, R6.2, V4.2; no longer Q14.3 (E), Q2.3 (E), R9.2
- net VCC: now also Q14.1 (C), Q2.1 (C), R8.1, R9.1, Q1.1 (C), Q11.1 (C), Q17.1 (C), Q19.1 (C), Q21.1 (C), Q24.3 (E), Q28.1 (C), Q29.1 (C), Q33.1 (C), Q34.1 (C), Q35.3 (E), Q42.3 (E), Q43.1 (C), Q44.1 (C), R15.1, R16.1, R19.1, R21.1, R23.1, R26.1, R27.1, R32.1, R33.1, R34.1, R39.1, R7.1; no longer R3.1, R5.1
- removed net BASE: D1.1 (A), D2.1 (A), Q14.2 (B), Q2.2 (B), R1.2, R2.1, R8.2, R9.1
- net IN_A: no longer names the net of Q12.2 (B)
- net IN_A: now also R10.2, Q10.3 (E), Q8.3 (E); no longer V2.1
- removed net IN_B: Q13.2 (B), Q7.2 (B), V3.1
- removed net OUT: D1.3 (K), Q2.1 (C), R3.2
- new net: Q39.3 (E), Q41.3 (E), Q43.2 (B), R33.2
- new net: D8.3 (K), Q35.2 (B), R27.2, R28.1
- new net: Q31.3 (E), Q32.3 (E), R28.2
- new net: Q1.3 (E), Q3.3 (E), R3.1
- new net: D6.3 (K), Q24.2 (B), R19.2, R20.1
- new net: Q18.3 (E), Q20.3 (E), Q22.3 (E), R20.2
- new net: D3.1 (A), Q15.2 (B), R11.2, R12.1
- new net: D1.1 (A), Q5.2 (B), R3.2, R4.1
- new net: D10.3 (K), Q42.2 (B), R34.2, R35.1
- new net: D11.1 (A), Q45.2 (B), R37.2, R38.1
- new net: D4.1 (A), Q16.2 (B), R13.2, R14.1
- new net: D7.1 (A), Q30.2 (B), R24.2, R25.1
- new net: Q11.2 (B), Q7.3 (E), Q9.3 (E), R9.2
- new net: Q43.3 (E), Q44.3 (E), R37.1
- new net: D5.1 (A), Q23.2 (B), R17.2, R18.1
- new net: D2.3 (K), Q14.2 (B), Q6.1 (C), R8.2
- new net: D8.1 (A), Q35.1 (C), Q40.2 (B), R31.1
- new net: D1.3 (K), Q13.2 (B), Q5.1 (C), R7.2
- new net: Q25.3 (E), Q26.3 (E), Q27.3 (E), Q28.2 (B), R23.2
- new net: Q17.3 (E), Q19.3 (E), Q21.3 (E), R17.1
- new net: Q37.3 (E), Q38.3 (E), Q40.3 (E), R35.2
- new net: Q28.3 (E), Q29.3 (E), R24.1
- new net: D9.3 (K), Q36.1 (C), Q44.2 (B), R32.2
- new net: Q11.3 (E), Q13.3 (E), R11.1
- new net: Q2.3 (E), Q4.3 (E), R5.1
- new net: Q33.3 (E), Q34.3 (E), R29.1
- new net: Q12.3 (E), Q14.3 (E), R13.1
- new net: D2.1 (A), Q6.2 (B), R5.2, R6.1
- new net: D9.1 (A), Q36.2 (B), R29.2, R30.1
- new net: D5.3 (K), Q23.1 (C), Q29.2 (B), R21.2
- new net A0: D3.3 (K), Q15.1 (C), Q19.2 (B), Q20.2 (B), Q25.2 (B), R15.2
- new net AND_EN: Q17.2 (B)
- new net B0: D4.3 (K), Q16.1 (C), Q21.2 (B), Q22.2 (B), Q26.2 (B), R16.2
- new net IN_A0: Q1.2 (B), Q7.2 (B), V2.1
- new net IN_B0: Q2.2 (B), Q8.2 (B), V3.1
- new net IN_C0: Q31.2 (B), Q33.2 (B), Q39.2 (B), V4.1
- new net IN_INV_A: Q3.2 (B), Q9.2 (B), R1.1
- new net IN_INV_B: Q10.2 (B), Q4.2 (B), R2.1
- new net OUT_C1: D10.1 (A), Q42.1 (C), R36.1
- new net OUT_P0: D7.3 (K), Q30.1 (C), Q32.2 (B), Q34.2 (B), Q41.2 (B), R26.2
- new net OUT_S0: D11.3 (K), Q45.1 (C), R39.2
- new net ~{IN_C_IS_0}: Q18.2 (B)
- new net ~{IN_C_IS_1}: Q37.2 (B)
- new net ~{OR_EN}: Q27.2 (B)
- new net ~{OUT_G0}: D6.1 (A), Q24.1 (C), Q38.2 (B), R22.1
Other:
- note added: ".param edge=1n"
- note added: ".param freq=1Mega"

Commit message: Full 16-bit ALU out of transistors.
The propagation delay seems to be pretty
good, actually:

~220ns at 125C and (thought the sim is still running)
~350ns at -25C

This is well within target for 400ns and
kind of surprising for a ripple-carry
implementation. However if it holds,
this makes things much easier on the
implementation.

BTW: ROL/ROR bit-forwarding is hooked
up incorrectly on the top, so that needs
to be fixed.

Also, only ADD is tested at the moment.
The rest should be easy as mostly can be
tested on the bit level.
Parts:
- removed D1, D10, D11, D2, D3, D4, D5, D6, D7, D8, D9: BAT54W, Package_TO_SOT_SMD:SOT-323_SC-70, symbol Diode:BAT54W
- removed Q1, Q11, Q12, Q13, Q14, Q15, Q16, Q17, Q19, Q2, Q21, Q23, Q28, Q29, Q3, Q30, Q33, Q34, Q36, Q4, Q43, Q44, Q45, Q5, Q6: 2N3904, Package_TO_SOT_SMD:SOT-23-3, symbol Simulation_SPICE:NPN
- removed Q10, Q18, Q20, Q22, Q24, Q25, Q26, Q27, Q31, Q32, Q35, Q37, Q38, Q39, Q40, Q41, Q42, Q7, Q8, Q9: 2N3906, Package_TO_SOT_SMD:SOT-23-3, symbol Simulation_SPICE:PNP
- removed R1, R2: 10k, Resistor_SMD:R_0603_1608Metric_Pad0.98x0.95mm_HandSolder, symbol Device:R_Small_US
- removed R10, R23, R33, R9: 520, Resistor_SMD:R_0603_1608Metric_Pad0.98x0.95mm_HandSolder, symbol Device:R_Small_US
- removed R11, R12, R13, R14, R17, R18, R19, R20, R24, R25, R27, R28, R29, R3, R30, R34, R35, R37, R38, R4, R5, R6: 220, Resistor_SMD:R_0603_1608Metric_Pad0.98x0.95mm_HandSolder, symbol Device:R_Small_US
- removed R15, R16, R21, R22, R26, R31, R32, R36, R39, R7, R8: 100, Resistor_SMD:R_0603_1608Metric_Pad0.98x0.95mm_HandSolder, symbol Device:R_Small_US
- added R377, R378, R379, R380, R381, R382, R383, R384, R761, R762, R763, R764, R765, R766, R767, R768, R769, R770, R771, R772, R773, R774, R775, R776, R777, R778, R779, R780, R781, R782, R783, R784: 1m, Resistor_SMD:R_0603_1608Metric_Pad0.98x0.95mm_HandSolder, symbol Device:R_Small_US
Connections:
- net A0: now also R377.2
- net B0: now also R381.2
- net IN_A0 renamed A
- net A: now also R377.1, R378.1, R379.1, R380.1, R761.1, R762.1, R763.1, R764.1, R769.1, R770.1, R771.1, R772.1, R773.1, R774.1, R775.1, R776.1
- net IN_B0 renamed B
- net B: now also R381.1, R382.1, R383.1, R384.1, R765.1, R766.1, R767.1, R768.1, R777.1, R778.1, R779.1, R780.1, R781.1, R782.1, R783.1, R784.1
- net IN_C0 renamed C_IN
- new net A1: R378.2
- new net A10: R771.2
- new net A11: R772.2
- new net A12: R773.2
- new net A13: R774.2
- new net A14: R775.2
- new net A15: R776.2
- new net A2: R379.2
- new net A3: R380.2
- new net A4: R761.2
- new net A5: R762.2
- new net A6: R763.2
- new net A7: R764.2
- new net A8: R769.2
- new net A9: R770.2
- new net B1: R382.2
- new net B10: R779.2
- new net B11: R780.2
- new net B12: R781.2
- new net B13: R782.2
- new net B14: R783.2
- new net B15: R784.2
- new net B2: R383.2
- new net B3: R384.2
- new net B4: R765.2
- new net B5: R766.2
- new net B6: R767.2
- new net B7: R768.2
- new net B8: R777.2
- new net B9: R778.2
Other:
- added sheet alu_4 (alu_4.kicad_sch)
- added sheet alu_5 (alu_4.kicad_sch)
- added sheet alu_6 (alu_4.kicad_sch)
- added sheet alu_7 (alu_4.kicad_sch)
- note added: ".param freq=0.25Mega"
- note removed: ".param freq=1Mega"

Commit message: Fixed ROL/ROR routing and added flags
This is not fully tested yet, but at least
complete in terms of functionality.

Latency still seems to be less than 350ns.
Parts:
- added D225, D226, D227, D228, D229, D230, D231, D232, D233, D234: BAT54W, Package_TO_SOT_SMD:SOT-323_SC-70, symbol Diode:BAT54W
- added Q913, Q914, Q915, Q918, Q919, Q920, Q921, Q922, Q923, Q924, Q925, Q926, Q927, Q928, Q929, Q930, Q931, Q932, Q933, Q934, Q935, Q936, Q937, Q938, Q939, Q940, Q941, Q942, Q943, Q946, Q947, Q948, Q949, Q950, Q951, Q954, Q955, Q956, Q961: 2N3904, Package_TO_SOT_SMD:SOT-23-3, symbol Simulation_SPICE:NPN
- added Q916, Q917, Q944, Q945, Q952, Q953, Q958, Q959, Q960: 2N3906, Package_TO_SOT_SMD:SOT-23-3, symbol Simulation_SPICE:PNP
- added R785, R786, R789, R790, R801, R802, R804, R805, R807, R808, R811, R812, R814, R815, R818, R819, R821, R822: 220, Resistor_SMD:R_0603_1608Metric_Pad0.98x0.95mm_HandSolder, symbol Device:R_Small_US
- added R787, R791, R803, R806, R809, R813, R816, R820, R823, R824, R825: 100, Resistor_SMD:R_0603_1608Metric_Pad0.98x0.95mm_HandSolder, symbol Device:R_Small_US
- added R788, R810, R817: 520, Resistor_SMD:R_0603_1608Metric_Pad0.98x0.95mm_HandSolder, symbol Device:R_Small_US
- added R792, R793, R794, R795, R796, R797, R798, R799, R800: 1m, Resistor_SMD:R_0603_1608Metric_Pad0.98x0.95mm_HandSolder, symbol Device:R_Small_US
Connections:
- net 0: now also Q915.3 (E), Q916.1 (C), Q917.1 (C), Q920.3 (E), Q923.3 (E), Q926.3 (E), Q943.3 (E), Q944.1 (C), Q945.1 (C), Q948.3 (E), Q951.3 (E), Q952.1 (C), Q953.1 (C), Q956.3 (E), Q958.1 (C), Q959.1 (C), Q961.3 (E), R786.2, R790.2, R792.2, R794.2, R795.2, R797.2, R799.2, R800.2, R802.2, R805.2, R808.2, R812.2, R815.2, R819.2, R824.2
- net A: now also V3.1; no longer V2.1
- net A15: now also Q941.2 (B), Q944.2 (B), Q949.2 (B), Q952.2 (B)
- net B: now also V4.1; no longer V3.1
- net B15: now also Q942.2 (B), Q945.2 (B)
- net C16: now also Q913.2 (B), Q916.2 (B)
- net C_IN: now also V2.1; no longer V4.1
- net S0: now also Q933.2 (B)
- net S1: now also Q934.2 (B)
- net S10: now also Q931.2 (B)
- net S11: now also Q932.2 (B)
- net S12: now also Q928.2 (B)
- net S13: now also Q927.2 (B)
- net S14: now also Q924.2 (B)
- net S2: now also Q935.2 (B)
- net S3: now also Q936.2 (B)
- net S4: now also Q937.2 (B)
- net S5: now also Q938.2 (B)
- net S6: now also Q939.2 (B)
- net S7: now also Q940.2 (B)
- net S8: now also Q929.2 (B)
- net S9: now also Q930.2 (B)
- net VCC: now also Q913.1 (C), Q914.1 (C), Q918.1 (C), Q919.1 (C), Q921.1 (C), Q922.1 (C), Q924.1 (C), Q925.1 (C), Q927.1 (C), Q928.1 (C), Q929.1 (C), Q930.1 (C), Q931.1 (C), Q932.1 (C), Q933.1 (C), Q934.1 (C), Q935.1 (C), Q936.1 (C), Q937.1 (C), Q938.1 (C), Q939.1 (C), Q940.1 (C), Q941.1 (C), Q942.1 (C), Q946.1 (C), Q947.1 (C), Q949.1 (C), Q950.1 (C), Q954.1 (C), Q955.1 (C), Q960.3 (E), R787.1, R788.1, R791.1, R793.2, R796.2, R798.2, R803.1, R806.1, R809.1, R810.1, R813.1, R816.1, R817.1, R820.1, R821.1, R825.1
- new net: Q924.3 (E), Q925.3 (E), Q927.3 (E), Q928.3 (E), Q929.3 (E), Q930.3 (E), Q931.3 (E), Q932.3 (E), Q933.3 (E), Q934.3 (E), Q935.3 (E), Q936.3 (E), Q937.3 (E), Q938.3 (E), Q939.3 (E), Q940.3 (E), R804.1
- new net: D230.1 (A), Q948.2 (B), R811.2, R812.1
- new net: D230.3 (K), Q948.1 (C), Q959.2 (B), R813.2
- new net: D227.1 (A), Q923.2 (B), R801.2, R802.1
- new net: D228.1 (A), Q926.2 (B), R804.2, R805.1
- new net: Q916.3 (E), Q917.3 (E), Q918.2 (B), R788.2
- new net: Q921.3 (E), Q922.3 (E), R801.1
- new net: D225.1 (A), Q915.2 (B), R785.2, R786.1
- new net: D225.3 (K), Q915.1 (C), Q919.2 (B), R787.2
- new net: Q954.3 (E), Q955.3 (E), R818.1
- new net: D232.1 (A), Q956.2 (B), R818.2, R819.1
- new net: Q946.3 (E), Q947.3 (E), R811.1
- new net: D231.1 (A), Q951.2 (B), R814.2, R815.1
- new net: D232.3 (K), Q956.1 (C), Q958.2 (B), R820.2
- new net: Q949.3 (E), Q950.3 (E), R814.1
- new net: D233.3 (K), Q960.2 (B), R821.2, R822.1
- new net: Q944.3 (E), Q945.3 (E), Q946.2 (B), R810.2
- new net: D226.1 (A), Q920.2 (B), R789.2, R790.1
- new net: D231.3 (K), Q951.1 (C), Q955.2 (B), R816.2
- new net: Q952.3 (E), Q953.3 (E), Q954.2 (B), R817.2
- new net: D227.3 (K), Q914.2 (B), Q917.2 (B), Q923.1 (C), R803.2
- new net: D233.1 (A), Q960.1 (C), R823.1
- new net: Q958.3 (E), Q959.3 (E), R822.2
- new net: Q918.3 (E), Q919.3 (E), R789.1
- new net: Q941.3 (E), Q942.3 (E), R807.1
- new net: D234.1 (A), Q961.2 (B), R823.2, R824.1
- new net: Q913.3 (E), Q914.3 (E), R785.1
- new net: D229.3 (K), Q943.1 (C), Q947.2 (B), R809.2
- new net: D229.1 (A), Q943.2 (B), R807.2, R808.1
- new net FLAG_S: Q925.2 (B), Q950.2 (B), Q953.2 (B)
- new net IN_ADD_EN: R796.1
- new net IN_AND_EN: R797.1
- new net IN_C_IS_1: R792.1
- new net IN_INV_A: Q922.2 (B), R795.1
- new net IN_INV_B: Q921.2 (B), R794.1
- new net IN_ROL_EN: R800.1
- new net IN_ROR_EN: R799.1
- new net ~{FLAG_C}: D226.3 (K), Q920.1 (C), R791.2
- new net ~{FLAG_V}: D234.3 (K), Q961.1 (C), R825.2
- new net ~{FLAG_Z}: D228.3 (K), Q926.1 (C), R806.2
- new net ~{IN_C_IS_0}: R793.1
- new net ~{IN_OR_EN}: R798.1

Commit message: Small ALU fix.
Parts:
- added R826: 1m, Resistor_SMD:R_0603_1608Metric_Pad0.98x0.95mm_HandSolder, symbol Device:R_Small_US
Connections:
- net C_IN: now also R826.2; no longer V2.1
- new net C: R826.1, V2.1
Changed lines of the file:
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@@
 	(wire
 		(pts
+			(xy 36.83 355.6) (xy 21.59 355.6)
+		)
+		(stroke
+			(width 0)
+			(type default)
+		)
+	)
+	(wire
+		(pts
 			(xy 262.89 300.99) (xy 270.51 300.99)
 		)
@@
 	(wire
 		(pts
+			(xy 44.45 77.47) (xy 52.07 77.47)
+		)
+		(stroke
+			(width 0)
+			(type default)
+		)
+	)
+	(wire
+		(pts
 			(xy 33.02 125.73) (xy 33.02 123.19)
 		)
@@
 	(wire
 		(pts
+			(xy 25.4 77.47) (xy 39.37 77.47)
+		)
+		(stroke
+			(width 0)
+			(type default)
+		)
+	)
+	(wire
+		(pts
 			(xy 314.96 236.22) (xy 317.5 236.22)
 		)
@@
 		)
 	)
+	(label "C_IN"
+		(at 46.99 77.47 0)
+		(effects
+			(font
+				(size 1.27 1.27)
+			)
+			(justify left bottom)
+		)
+	)
 	(label "A5"
 		(at 46.99 100.33 0)
@@
 		)
 	)
+	(label "C_IN"
+		(at 31.75 355.6 0)
+		(effects
+			(font
+				(size 1.27 1.27)
+			)
+			(justify left bottom)
+		)
+	)
 	(label "A10"
 		(at 31.75 387.35 0)
@@
 		)
 	)
-	(label "C_IN"
+	(label "C"
 		(at 41.91 44.45 0)
 		(effects
@@
 		)
 	)
+	(label "C"
+		(at 27.94 77.47 0)
+		(effects
+			(font
+				(size 1.27 1.27)
+			)
+			(justify left bottom)
+		)
+	)
 	(label "B10"
 		(at 60.96 387.35 0)
@@
 		)
 	)
+	(hierarchical_label "C_IN"
+		(shape input)
+		(at 21.59 355.6 180)
+		(effects
+			(font
+				(size 1.27 1.27)
+			)
+			(justify right)
+		)
+	)
 	(hierarchical_label "A0"
 		(shape input)
@@
 					(unit 1)
 				)
+			)
+		)
+	)
+	(symbol
+		(lib_id "Device:R_Small_US")
+		(at 41.91 77.47 90)
+		(unit 1)
+		(exclude_from_sim no)
+		(in_bom no)
+		(on_board no)
+		(dnp no)
+		(property "Reference" "R826"
+			(at 41.91 71.12 90)
+			(effects
+				(font
+					(size 1.27 1.27)
+				)
+				(hide yes)
+			)
+		)
+		(property "Value" "1m"
+			(at 36.83 76.2 90)
+			(effects
+				(font
+					(size 1.27 1.27)
+				)
+			)
+		)
+		(property "Footprint" "Resistor_SMD:R_0603_1608Metric_Pad0.98x0.95mm_HandSolder"
+			(at 41.91 77.47 0)
+			(effects
+				(font
+					(size 1.27 1.27)
+				)
+				(hide yes)
+			)
+		)
+		(property "Datasheet" "~"
+			(at 41.91 77.47 0)
+			(effects
+				(font
+					(size 1.27 1.27)
+				)
+				(hide yes)
+			)
+		)
+		(property "Description" "Resistor, small US symbol"
+			(at 41.91 77.47 0)
+			(effects
+				(font
+					(size 1.27 1.27)
+				)
+				(hide yes)
+			)
+		)
+		(pin "1"
+		)
+		(pin "2"
+		)
+		(instances
+			(project "alu"
+				(path "/ed92c5aa-463d-470b-a4b4-8d1a1cd780d2"
+					(reference "R826")
+					(unit 1)
+				)

Commit message: Some fixes to the ALU schematics
Parts:
- D225, D226, D227, D228, D229, D230, D231, D232, D233, D234: value BAT54W -> BAT54LT1G; footprint Package_TO_SOT_SMD:SOT-323_SC-70 -> Package_TO_SOT_SMD:SOT-23-3; symbol Diode:BAT54W -> TCOMP:BAT54LT1G
- Q913, Q914, Q915, Q918, Q919, Q920, Q921, Q922, Q923, Q924, Q925, Q926, Q927, Q928, Q929, Q930, Q931, Q932, Q933, Q934, Q935, Q936, Q937, Q938, Q939, Q940, Q941, Q942, Q943, Q946, Q947, Q948, Q949, Q950, Q951, Q954, Q955, Q956, Q961: symbol Simulation_SPICE:NPN -> TCOMP:2N3904
- Q916, Q917, Q944, Q945, Q952, Q953, Q958, Q959, Q960: symbol Simulation_SPICE:PNP -> TCOMP:2N3906
- V1, V2, V3, V4: now left out of the parts list
Connections:
- net 0 renamed GND
