File: modules/alu/bit_logic.kicad_sch (KiCad schematic)
At the start: 103 parts, among them Q257 2N3904, Q258 2N3904, Q259 2N3904, Q260 2N3904, Q261 2N3904, Q262 2N3904, Q263 2N3904, Q264 2N3904, Q265 2N3906, Q266 2N3906, Q267 2N3906, Q268 2N3906, Q269 2N3904, Q270 2N3904, Q271 2N3904, Q272 2N3906, Q273 2N3904, Q274 2N3904, Q275 2N3906, Q276 2N3904, Q277 2N3904, Q278 2N3904, Q279 2N3904, Q280 2N3904, Q281 2N3906, Q282 2N3904, Q283 2N3906, Q284 2N3904, Q285 2N3906, Q286 2N3904, Q287 2N3906, Q288 2N3906, Q289 2N3906, Q290 2N3904, Q291 2N3906, Q292 2N3906, Q293 2N3906, Q294 2N3906, Q295 2N3904, Q296 2N3906, Q297 2N3906, Q298 2N3906, Q299 2N3906, Q300 2N3904, Q301 2N3904, Q302 2N3904, Q303 2N3904, Q304 2N3904, Q305 2N3904, Q306 2N3904

Commit message: Fixed ROL/ROR routing and added flags
This is not fully tested yet, but at least
complete in terms of functionality.

Latency still seems to be less than 350ns.
Parts:
- renumbered D65 to D121, D66 to D122, D67 to D123, D68 to D124, D69 to D125, D70 to D126, D71 to D127, D72 to D128, D73 to D129, D74 to D130, D75 to D131, D76 to D132, Q257 to Q485, Q258 to Q486, Q259 to Q487, Q260 to Q488, Q261 to Q489, Q262 to Q490, Q263 to Q491, Q264 to Q492, Q265 to Q493, Q266 to Q494, Q267 to Q495, Q268 to Q496, Q269 to Q497, Q270 to Q498, Q271 to Q499, Q272 to Q500, Q273 to Q501, Q274 to Q502, Q275 to Q503, Q276 to Q504, Q277 to Q505, Q278 to Q506, Q279 to Q507, Q280 to Q508, Q281 to Q509, Q282 to Q510, Q283 to Q511, Q284 to Q512, Q285 to Q513, Q286 to Q514, Q287 to Q515, Q288 to Q516, Q289 to Q517, Q290 to Q518, Q291 to Q519, Q292 to Q520, Q293 to Q521, Q294 to Q522, Q295 to Q523, Q296 to Q524, Q297 to Q525, Q298 to Q526, Q299 to Q527, Q300 to Q528, Q301 to Q529, Q302 to Q530, Q303 to Q531, Q304 to Q532, Q305 to Q533, Q306 to Q534, R213 to R409, R214 to R410, R215 to R411, R216 to R412, R217 to R413, R218 to R414, R219 to R415, R220 to R416, R221 to R417, R222 to R418, R223 to R419, R224 to R420, R225 to R421, R226 to R422, R227 to R423, R228 to R424, R229 to R425, R230 to R426, R231 to R427, R232 to R428, R233 to R429, R234 to R430, R235 to R431, R236 to R432, R237 to R433, R238 to R434, R239 to R435, R240 to R436, R241 to R437, R242 to R438, R243 to R439, R244 to R440, R245 to R441, R246 to R442, R247 to R443, R248 to R444, R249 to R445, R250 to R446, R251 to R447, R252 to R448, R253 to R449

Commit message: Small ALU fix.
Parts:
- removed R430: 100, Resistor_SMD:R_0603_1608Metric_Pad0.98x0.95mm_HandSolder, symbol Device:R_Small_US
- added R46: 100, Resistor_SMD:R_0603_1608Metric_Pad0.98x0.95mm_HandSolder, symbol Device:R_Small_US
Connections:
- net OUT_S: now also D127.1 (A), Q509.1 (C), R431.1; no longer D132.3 (K), Q534.1 (C), R449.2
- net at D127.3 (K), Q509.2 (B): now also R449.2, R46.1; no longer R429.2
- net at D126.3 (K), Q508.1 (C): now also Q519.2 (B), R429.2
- new net: D132.3 (K), Q534.1 (C), R46.2
Other:
- note added: "AND with extra enabler for "GENERATE" generation"
- note added: "AND-OR to mux in ROR/ROR"
- note added: "XOR to generate SUM"
- note added: "XOR to invert A"
- note added: "XOR to invert B"
- note added: "XOR with extra enables for "PROPAGATE" generation"
- moved on the sheet: D121, D122, D123, D124, D125, D126, D127, D128, D129, D130, D131, D132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

Commit message: Moved carry generation into ALU bit-cell.
Parts:
- added D251, D252: BAT54W, Package_TO_SOT_SMD:SOT-323_SC-70, symbol Diode:BAT54W
- added Q1017, Q1018, Q1023: 2N3906, Package_TO_SOT_SMD:SOT-23-3, symbol Simulation_SPICE:PNP
- added Q1019, Q1020, Q1021, Q1022: 2N3904, Package_TO_SOT_SMD:SOT-23-3, symbol Simulation_SPICE:NPN
- added R875: 520, Resistor_SMD:R_0603_1608Metric_Pad0.98x0.95mm_HandSolder, symbol Device:R_Small_US
- added R876, R877: 220, Resistor_SMD:R_0603_1608Metric_Pad0.98x0.95mm_HandSolder, symbol Device:R_Small_US
- added R878, R879, R880: 100, Resistor_SMD:R_0603_1608Metric_Pad0.98x0.95mm_HandSolder, symbol Device:R_Small_US
- renumbered R46 to R430
Connections:
- net 0: now also Q1017.1 (C), Q1018.1 (C), Q1022.3 (E), R877.2, R880.2
- net IN_C: now also Q1018.2 (B)
- net OUT_G: now also Q1020.2 (B)
- net OUT_P: now also Q1017.2 (B)
- net VCC: now also Q1019.1 (C), Q1020.1 (C), Q1021.1 (C), Q1023.3 (E), R875.1, R878.1
- new net: D251.3 (K), Q1022.1 (C), R879.2
- new net: D251.1 (A), Q1022.2 (B), R876.2, R877.1
- new net: Q1019.3 (E), Q1020.3 (E), Q1021.3 (E), R876.1
- new net: D252.3 (K), Q1023.2 (B), R878.2, R879.1
- new net: Q1017.3 (E), Q1018.3 (E), Q1019.2 (B), R875.2
- new net IN_C_IS_1: Q1021.2 (B)
- new net OUT_C: D252.1 (A), Q1023.1 (C), R880.1
Other:
- note added: "AND-OR gate to implement CARRY"
- moved on the sheet: D123, D126, D127, D132, Q491, Q492, Q497, Q500, Q503, Q506, Q507, Q508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

Commit message: Some small ALU changes (need review!)
Connections:
- net XX: now reaches Q500.3 (E), Q503.3 (E), Q506.2 (B), R420.2
- net XX: now also Q1019.2 (B)
- net at Q1017.3 (E), Q1018.3 (E), R875.2: no longer Q1019.2 (B)
Changed lines of the file:
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@@
 	)
 	(junction
+		(at 127 295.91)
+		(diameter 0)
+		(color 0 0 0 0)
+	)
+	(junction
 		(at 83.82 356.87)
 		(diameter 0)
@@
 	)
 	(junction
-		(at 469.9 327.66)
-		(diameter 0)
-		(color 0 0 0 0)
-	)
-	(junction
 		(at 127 250.19)
 		(diameter 0)
@@
 	(wire
 		(pts
-			(xy 469.9 327.66) (xy 472.44 327.66)
-		)
-		(stroke
-			(width 0)
-			(type default)
-		)
-	)
-	(wire
-		(pts
 			(xy 189.23 27.94) (xy 189.23 31.75)
 		)
@@
 	(wire
 		(pts
+			(xy 127 271.78) (xy 154.94 271.78)
+		)
+		(stroke
+			(width 0)
+			(type default)
+		)
+	)
+	(wire
+		(pts
 			(xy 107.95 288.29) (xy 107.95 295.91)
 		)
@@
 	(wire
 		(pts
+			(xy 472.44 327.66) (xy 472.44 323.85)
+		)
+		(stroke
+			(width 0)
+			(type default)
+		)
+	)
+	(wire
+		(pts
 			(xy 354.33 83.82) (xy 354.33 161.29)
 		)
@@
 	(wire
 		(pts
-			(xy 119.38 295.91) (xy 138.43 295.91)
+			(xy 119.38 295.91) (xy 127 295.91)
 		)
 		(stroke
@@
 	(wire
 		(pts
+			(xy 433.07 323.85) (xy 472.44 323.85)
+		)
+		(stroke
+			(width 0)
+			(type default)
+		)
+	)
+	(wire
+		(pts
 			(xy 405.13 161.29) (xy 415.29 161.29)
 		)
@@
 	(wire
 		(pts
+			(xy 127 295.91) (xy 138.43 295.91)
+		)
+		(stroke
+			(width 0)
+			(type default)
+		)
+	)
+	(wire
+		(pts
 			(xy 237.49 279.4) (xy 260.35 279.4)
 		)
@@
 	(wire
 		(pts
+			(xy 127 295.91) (xy 127 271.78)
+		)
+		(stroke
+			(width 0)
+			(type default)
+		)
+	)
+	(wire
+		(pts
 			(xy 168.91 384.81) (xy 168.91 389.89)
 		)
@@
 		)
 	)
+	(label "XX"
+		(at 443.23 323.85 0)
+		(effects
+			(font
+				(size 1.27 1.27)
+			)
+			(justify left bottom)
+		)
+	)
 	(label "OUT_G"
 		(at 360.68 213.36 0)
@@
 		(effects
 			(font
+				(size 1.27 1.27)
+			)
+			(justify left bottom)
+		)
+	)
+	(label "XX"
+		(at 138.43 271.78 0)
+		(effects
+			(font

Commit message: Some fixes to the ALU schematics
Parts:
- added J1: PCIe_4x_edge, tcomp:BUS_PCIexpress_x4, symbol TCOMP:PCIe_4x_edge
- added R1: 0, Resistor_SMD:R_0603_1608Metric_Pad0.98x0.95mm_HandSolder, symbol Device:R_Small_US
- D10: renamed from D122; value BAT54W -> BAT54LT1G; footprint Package_TO_SOT_SMD:SOT-323_SC-70 -> Package_TO_SOT_SMD:SOT-23-3; symbol Diode:BAT54W -> TCOMP:BAT54LT1G
- D11: renamed from D123; value BAT54W -> BAT54LT1G; footprint Package_TO_SOT_SMD:SOT-323_SC-70 -> Package_TO_SOT_SMD:SOT-23-3; symbol Diode:BAT54W -> TCOMP:BAT54LT1G
- D12: renamed from D124; value BAT54W -> BAT54LT1G; footprint Package_TO_SOT_SMD:SOT-323_SC-70 -> Package_TO_SOT_SMD:SOT-23-3; symbol Diode:BAT54W -> TCOMP:BAT54LT1G
- D13: renamed from D125; value BAT54W -> BAT54LT1G; footprint Package_TO_SOT_SMD:SOT-323_SC-70 -> Package_TO_SOT_SMD:SOT-23-3; symbol Diode:BAT54W -> TCOMP:BAT54LT1G
- D14: renamed from D126; value BAT54W -> BAT54LT1G; footprint Package_TO_SOT_SMD:SOT-323_SC-70 -> Package_TO_SOT_SMD:SOT-23-3; symbol Diode:BAT54W -> TCOMP:BAT54LT1G
- D15: renamed from D127; value BAT54W -> BAT54LT1G; footprint Package_TO_SOT_SMD:SOT-323_SC-70 -> Package_TO_SOT_SMD:SOT-23-3; symbol Diode:BAT54W -> TCOMP:BAT54LT1G
- D16: renamed from D128; value BAT54W -> BAT54LT1G; footprint Package_TO_SOT_SMD:SOT-323_SC-70 -> Package_TO_SOT_SMD:SOT-23-3; symbol Diode:BAT54W -> TCOMP:BAT54LT1G
- D17: renamed from D129; value BAT54W -> BAT54LT1G; footprint Package_TO_SOT_SMD:SOT-323_SC-70 -> Package_TO_SOT_SMD:SOT-23-3; symbol Diode:BAT54W -> TCOMP:BAT54LT1G
- D18: renamed from D130; value BAT54W -> BAT54LT1G; footprint Package_TO_SOT_SMD:SOT-323_SC-70 -> Package_TO_SOT_SMD:SOT-23-3; symbol Diode:BAT54W -> TCOMP:BAT54LT1G
- D19: renamed from D131; value BAT54W -> BAT54LT1G; footprint Package_TO_SOT_SMD:SOT-323_SC-70 -> Package_TO_SOT_SMD:SOT-23-3; symbol Diode:BAT54W -> TCOMP:BAT54LT1G
- D20: renamed from D132; value BAT54W -> BAT54LT1G; footprint Package_TO_SOT_SMD:SOT-323_SC-70 -> Package_TO_SOT_SMD:SOT-23-3; symbol Diode:BAT54W -> TCOMP:BAT54LT1G
- D235: renamed from D251; value BAT54W -> BAT54LT1G; footprint Package_TO_SOT_SMD:SOT-323_SC-70 -> Package_TO_SOT_SMD:SOT-23-3; symbol Diode:BAT54W -> TCOMP:BAT54LT1G
- D236: renamed from D252; value BAT54W -> BAT54LT1G; footprint Package_TO_SOT_SMD:SOT-323_SC-70 -> Package_TO_SOT_SMD:SOT-23-3; symbol Diode:BAT54W -> TCOMP:BAT54LT1G
- D9: renamed from D121; value BAT54W -> BAT54LT1G; footprint Package_TO_SOT_SMD:SOT-323_SC-70 -> Package_TO_SOT_SMD:SOT-23-3; symbol Diode:BAT54W -> TCOMP:BAT54LT1G
- Q29: renamed from Q485; symbol Simulation_SPICE:NPN -> TCOMP:2N3904
- Q30: renamed from Q486; symbol Simulation_SPICE:NPN -> TCOMP:2N3904
- Q31: renamed from Q487; symbol Simulation_SPICE:NPN -> TCOMP:2N3904
- Q32: renamed from Q488; symbol Simulation_SPICE:NPN -> TCOMP:2N3904
- Q33: renamed from Q489; symbol Simulation_SPICE:NPN -> TCOMP:2N3904
- Q34: renamed from Q490; symbol Simulation_SPICE:NPN -> TCOMP:2N3904
- Q35: renamed from Q491; symbol Simulation_SPICE:NPN -> TCOMP:2N3904
- Q36: renamed from Q492; symbol Simulation_SPICE:NPN -> TCOMP:2N3904
- Q37: renamed from Q493; symbol Simulation_SPICE:PNP -> TCOMP:2N3906
- Q38: renamed from Q494; symbol Simulation_SPICE:PNP -> TCOMP:2N3906
- Q39: renamed from Q495; symbol Simulation_SPICE:PNP -> TCOMP:2N3906
- Q40: renamed from Q496; symbol Simulation_SPICE:PNP -> TCOMP:2N3906
- Q41: renamed from Q497; symbol Simulation_SPICE:NPN -> TCOMP:2N3904
- Q42: renamed from Q498; symbol Simulation_SPICE:NPN -> TCOMP:2N3904
- Q43: renamed from Q499; symbol Simulation_SPICE:NPN -> TCOMP:2N3904
- Q44: renamed from Q500; symbol Simulation_SPICE:PNP -> TCOMP:2N3906
- Q45: renamed from Q501; symbol Simulation_SPICE:NPN -> TCOMP:2N3904
- Q46: renamed from Q502; symbol Simulation_SPICE:NPN -> TCOMP:2N3904
- Q47: renamed from Q503; symbol Simulation_SPICE:PNP -> TCOMP:2N3906
- Q48: renamed from Q504; symbol Simulation_SPICE:NPN -> TCOMP:2N3904
- Q49: renamed from Q505; symbol Simulation_SPICE:NPN -> TCOMP:2N3904
- Q50: renamed from Q506; symbol Simulation_SPICE:NPN -> TCOMP:2N3904
- Q51: renamed from Q507; symbol Simulation_SPICE:NPN -> TCOMP:2N3904
- Q52: renamed from Q508; symbol Simulation_SPICE:NPN -> TCOMP:2N3904
- Q53: renamed from Q509; symbol Simulation_SPICE:PNP -> TCOMP:2N3906
- Q54: renamed from Q510; symbol Simulation_SPICE:NPN -> TCOMP:2N3904
- Q55: renamed from Q511; symbol Simulation_SPICE:PNP -> TCOMP:2N3906
- Q56: renamed from Q512; symbol Simulation_SPICE:NPN -> TCOMP:2N3904
- Q57: renamed from Q513; symbol Simulation_SPICE:PNP -> TCOMP:2N3906
- Q58: renamed from Q514; symbol Simulation_SPICE:NPN -> TCOMP:2N3904
- Q59: renamed from Q515; symbol Simulation_SPICE:PNP -> TCOMP:2N3906
- Q60: renamed from Q516; symbol Simulation_SPICE:PNP -> TCOMP:2N3906
- Q61: renamed from Q517; symbol Simulation_SPICE:PNP -> TCOMP:2N3906
- Q62: renamed from Q518; symbol Simulation_SPICE:NPN -> TCOMP:2N3904
- Q63: renamed from Q519; symbol Simulation_SPICE:PNP -> TCOMP:2N3906
- Q64: renamed from Q520; symbol Simulation_SPICE:PNP -> TCOMP:2N3906
- Q65: renamed from Q521; symbol Simulation_SPICE:PNP -> TCOMP:2N3906
- Q66: renamed from Q522; symbol Simulation_SPICE:PNP -> TCOMP:2N3906
- Q67: renamed from Q523; symbol Simulation_SPICE:NPN -> TCOMP:2N3904
- Q68: renamed from Q524; symbol Simulation_SPICE:PNP -> TCOMP:2N3906
- Q69: renamed from Q525; symbol Simulation_SPICE:PNP -> TCOMP:2N3906
- Q70: renamed from Q526; symbol Simulation_SPICE:PNP -> TCOMP:2N3906
- Q71: renamed from Q527; symbol Simulation_SPICE:PNP -> TCOMP:2N3906
- Q72: renamed from Q528; symbol Simulation_SPICE:NPN -> TCOMP:2N3904
- Q73: renamed from Q529; symbol Simulation_SPICE:NPN -> TCOMP:2N3904
- Q74: renamed from Q530; symbol Simulation_SPICE:NPN -> TCOMP:2N3904
- Q75: renamed from Q531; symbol Simulation_SPICE:NPN -> TCOMP:2N3904
- Q76: renamed from Q532; symbol Simulation_SPICE:NPN -> TCOMP:2N3904
- Q77: renamed from Q533; symbol Simulation_SPICE:NPN -> TCOMP:2N3904
- Q78: renamed from Q534; symbol Simulation_SPICE:NPN -> TCOMP:2N3904
- Q957: renamed from Q1017; symbol Simulation_SPICE:PNP -> TCOMP:2N3906; now not fitted
- Q962: renamed from Q1018; symbol Simulation_SPICE:PNP -> TCOMP:2N3906; now not fitted
- Q963: renamed from Q1019; symbol Simulation_SPICE:NPN -> TCOMP:2N3904
- Q964: renamed from Q1020; symbol Simulation_SPICE:NPN -> TCOMP:2N3904
- Q965: renamed from Q1021; symbol Simulation_SPICE:NPN -> TCOMP:2N3904
- Q966: renamed from Q1022; symbol Simulation_SPICE:NPN -> TCOMP:2N3904
- Q967: renamed from Q1023; symbol Simulation_SPICE:PNP -> TCOMP:2N3906
- R827: renamed from R875; now not fitted
- renumbered R409 to R25, R410 to R26, R411 to R27, R412 to R28, R413 to R29, R414 to R30, R415 to R31, R416 to R32, R417 to R33, R418 to R34, R419 to R35, R420 to R36, R421 to R37, R422 to R38, R423 to R39, R424 to R40, R425 to R41, R426 to R42, R427 to R43, R428 to R44, R429 to R45, R430 to R46, R431 to R47, R432 to R48, R433 to R49, R434 to R50, R435 to R51, R436 to R52, R437 to R53, R438 to R54, R439 to R55, R440 to R56, R441 to R57, R442 to R58, R443 to R59, R444 to R60, R445 to R61, R446 to R62, R447 to R63, R448 to R64, R449 to R65, R876 to R828, R877 to R829, R878 to R830, R879 to R831, R880 to R832
Connections:
- net IN_A: now also J1.A12 (Pin_a12)
- net IN_AND_EN: now also J1.A17 (Pin_a17)
- net IN_B: now also J1.A13 (Pin_a13)
- net IN_C: now also J1.A14 (Pin_a14)
- net IN_C_IS_1: now also J1.A20 (Pin_a20)
- net IN_INV_A: now also J1.A15 (Pin_a15)
- net IN_INV_B: now also J1.A16 (Pin_a16)
- net OUT_A: now also J1.A21 (Pin_a21)
- net OUT_C: now also J1.A22 (Pin_a22)
- net OUT_G: now also J1.A24 (Pin_a24)
- net OUT_P: now also J1.A25 (Pin_a25)
- net OUT_S: now also J1.A23 (Pin_a23)
- net VCC: now also J1.A10 (Pin_a10), J1.A11 (Pin_a11)
- net XX: now also R1.1; no longer Q963.2 (B)
- net ~{IN_C_IS_0}: now also J1.A19 (Pin_a19)
- net ~{IN_OR_EN}: now also J1.A18 (Pin_a18)
- net at Q957.3 (E), Q962.3 (E), R827.2: now also Q963.2 (B), R1.2
- net 0 renamed GND
- net GND: now also J1.B10 (Pin_b10), J1.B11 (Pin_b11), J1.B12 (Pin_b12), J1.B13 (Pin_b13), J1.B14 (Pin_b14), J1.B15 (Pin_b15), J1.B16 (Pin_b16), J1.B17 (Pin_b17), J1.B18 (Pin_b18), J1.B19 (Pin_b19), J1.B20 (Pin_b20), J1.B21 (Pin_b21), J1.B22 (Pin_b22), J1.B23 (Pin_b23), J1.B24 (Pin_b24), J1.B25 (Pin_b25), J1.B26 (Pin_b26), J1.B27 (Pin_b27), J1.B28 (Pin_b28), J1.B29 (Pin_b29), J1.B30 (Pin_b30), J1.B31 (Pin_b31), J1.B32 (Pin_b32)
Other:
- note added: "Replicated implementation of the (OUT_P and IN_C) term"
