File: modules/alu/bit_logic/bit_logic.kicad_sch (KiCad schematic)
At the start: 120 parts, among them J1 PCIe_4x_edge, Q29 2N3904, Q30 2N3904, Q31 2N3904, Q32 2N3904, Q33 2N3904, Q34 2N3904, Q35 2N3904, Q36 2N3904, Q37 2N3906, Q38 2N3906, Q39 2N3906, Q40 2N3906, Q41 2N3904, Q42 2N3904, Q43 2N3904, Q44 2N3906, Q45 2N3904, Q46 2N3904, Q47 2N3906, Q48 2N3904, Q49 2N3904, Q50 2N3904, Q51 2N3904, Q52 2N3904, Q53 2N3906, Q54 2N3904, Q55 2N3906, Q56 2N3904, Q57 2N3906, Q58 2N3904, Q59 2N3906, Q60 2N3906, Q61 2N3906, Q62 2N3904, Q63 2N3906, Q64 2N3906, Q65 2N3906, Q66 2N3906, Q67 2N3904, Q68 2N3906, Q69 2N3906, Q70 2N3906, Q71 2N3906, Q72 2N3904, Q73 2N3904, Q74 2N3904, Q75 2N3904, Q76 2N3904, Q77 2N3904, Q78 2N3904, Q957 2N3906, Q962 2N3906, Q963 2N3904, Q964 2N3904, Q965 2N3904, Q966 2N3904, Q967 2N3906

Commit message: Pretty good progress on bit-logic for ALU.
Parts:
- renumbered D11 to D1, D20 to D10, D15 to D11, D19 to D12, D235 to D13, D236 to D14, D9 to D2, D10 to D3, D14 to D4, D12 to D5, D13 to D6, D16 to D7, D17 to D8, D18 to D9, Q35 to Q1, Q44 to Q10, Q47 to Q11, Q37 to Q12, Q38 to Q13, Q39 to Q14, Q40 to Q15, Q50 to Q16, Q51 to Q17, Q42 to Q18, Q43 to Q19, Q36 to Q2, Q45 to Q20, Q46 to Q21, Q52 to Q22, Q48 to Q23, Q49 to Q24, Q60 to Q25, Q61 to Q26, Q63 to Q27, Q65 to Q28, Q54 to Q29, Q29 to Q3, Q68 to Q30, Q55 to Q31, Q56 to Q32, Q70 to Q33, Q57 to Q34, Q58 to Q35, Q72 to Q36, Q59 to Q37, Q74 to Q38, Q62 to Q39, Q30 to Q4, Q76 to Q40, Q64 to Q41, Q66 to Q42, Q67 to Q43, Q78 to Q44, Q69 to Q45, Q71 to Q46, Q53 to Q47, Q73 to Q48, Q75 to Q49, Q31 to Q5, Q77 to Q50, Q957 to Q51, Q962 to Q52, Q963 to Q53, Q964 to Q54, Q965 to Q55, Q966 to Q56, Q967 to Q57, Q32 to Q6, Q41 to Q7, Q33 to Q8, Q34 to Q9, R31 to R1, R36 to R10, R33 to R11, R34 to R12, R43 to R13, R44 to R14, R37 to R15, R38 to R16, R39 to R17, R40 to R18, R45 to R19, R32 to R2, R41 to R20, R42 to R21, R52 to R22, R54 to R23, R59 to R24, R48 to R25, R49 to R26, R50 to R27, R51 to R28, R53 to R29, R25 to R3, R62 to R30, R63 to R31, R55 to R32, R56 to R33, R57 to R34, R58 to R35, R65 to R36, R46 to R37, R47 to R38, R60 to R39, R26 to R4, R61 to R40, R64 to R41, R1 to R42, R827 to R43, R828 to R44, R829 to R45, R830 to R46, R831 to R47, R832 to R48, R27 to R5, R28 to R6, R35 to R7, R29 to R8, R30 to R9
Connections:
- net GND: now also J1.A10 (Pin_a10), J1.A11 (Pin_a11), J1.A12 (Pin_a12), J1.A13 (Pin_a13), J1.A14 (Pin_a14), J1.A15 (Pin_a15), J1.A16 (Pin_a16), J1.A17 (Pin_a17), J1.A18 (Pin_a18), J1.A19 (Pin_a19), J1.A20 (Pin_a20), J1.A21 (Pin_a21), J1.A22 (Pin_a22), J1.A23 (Pin_a23), J1.A24 (Pin_a24), J1.A25 (Pin_a25), J1.A26 (Pin_a26), J1.A27 (Pin_a27), J1.A28 (Pin_a28), J1.A29 (Pin_a29), J1.A30 (Pin_a30), J1.A31 (Pin_a31), J1.A32 (Pin_a32); no longer J1.B10 (Pin_b10), J1.B11 (Pin_b11), J1.B12 (Pin_b12), J1.B13 (Pin_b13), J1.B14 (Pin_b14), J1.B15 (Pin_b15), J1.B16 (Pin_b16), J1.B17 (Pin_b17), J1.B18 (Pin_b18), J1.B19 (Pin_b19), J1.B20 (Pin_b20), J1.B21 (Pin_b21), J1.B22 (Pin_b22), J1.B23 (Pin_b23), J1.B24 (Pin_b24), J1.B25 (Pin_b25), J1.B26 (Pin_b26), J1.B27 (Pin_b27), J1.B28 (Pin_b28), J1.B29 (Pin_b29), J1.B30 (Pin_b30), J1.B31 (Pin_b31), J1.B32 (Pin_b32)
- net IN_A: now also J1.B14 (Pin_b14); no longer J1.A12 (Pin_a12)
- net IN_ADD_EN: now also J1.B24 (Pin_b24)
- net IN_AND_EN: now also J1.B19 (Pin_b19); no longer J1.A17 (Pin_a17)
- net IN_A_NEXT: now also J1.B26 (Pin_b26)
- net IN_A_PREV: now also J1.B25 (Pin_b25)
- net IN_B: now also J1.B13 (Pin_b13); no longer J1.A13 (Pin_a13)
- net IN_C: now also J1.B30 (Pin_b30); no longer J1.A14 (Pin_a14)
- net IN_C_IS_1: now also J1.B20 (Pin_b20); no longer J1.A20 (Pin_a20)
- net IN_INV_A: now also J1.B17 (Pin_b17); no longer J1.A15 (Pin_a15)
- net IN_INV_B: now also J1.B15 (Pin_b15); no longer J1.A16 (Pin_a16)
- net IN_ROL_EN: now also J1.B22 (Pin_b22)
- net IN_ROR_EN: now also J1.B23 (Pin_b23)
- net OUT_A: now also J1.B27 (Pin_b27); no longer J1.A21 (Pin_a21)
- net OUT_C: now also J1.B28 (Pin_b28); no longer J1.A22 (Pin_a22)
- net OUT_G: now also J1.B32 (Pin_b32); no longer J1.A24 (Pin_a24)
- net OUT_P: now also J1.B29 (Pin_b29); no longer J1.A25 (Pin_a25)
- net OUT_S: now also J1.B31 (Pin_b31); no longer J1.A23 (Pin_a23)
- net VCC: now also J1.B10 (Pin_b10), J1.B11 (Pin_b11); no longer J1.A10 (Pin_a10), J1.A11 (Pin_a11)
- net ~{IN_C_IS_0}: now also J1.B16 (Pin_b16); no longer J1.A19 (Pin_a19)
- net ~{IN_OR_EN}: now also J1.B18 (Pin_b18); no longer J1.A18 (Pin_a18)
Other:
- moved on the sheet: R29
